Commit message: added slam_toolbox and nav2

File: description/robot_core.xacro (robot description, xacro)
@@ -5,4 +5,12 @@
     <!-- Base Link -->
     <link name="base_link">
+    </link>
+    <!-- this is needed for slam -->
+    <joint name="base_footprint_joint" type="fixed">
+        <parent link="base_link"/>
+        <child link="base_footprint"/>
+        <origin xyz="0.0 0.0 0.0" rpy="0.0 0.0 0.0"/>
+    </joint>
+    <link name="base_footprint">
     </link>
     <!-- Chassis link-->
